File: Hardware/SparkFun_CP2103_Breakout.sch (EAGLE design)
At the start: 17 parts, among them U1 CP2103, X1 USBPTH

Commit message: Updating hardware files
Other:
- note added: "v11"
Changed lines of the file:
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@@
 <sheet>
 <plain>
+<text x="241.3" y="7.62" size="1.27" layer="94">v11</text>
 </plain>
 <instances>
